Commit message: version 0.0.1 release, fixed name spaces

File: src/yamaro/output.urdf (robot description, URDF)
Before this commit: robot drone, 8 links, 7 joints
Links:
- removed link arm_0_link
- removed link arm_1_link
- removed link arm_2_link
- removed link arm_3_link
- removed link arm_4_link
- removed link arm_5_link
- removed link base_link
- added link arm_left_link; collision box size=1.2 0.1 0.1; visual box size=1.2 0.1 0.1
- added link arm_right_link; collision box size=1.0 0.1 0.1; visual box size=1.0 0.1 0.1
Joints:
- removed joint arm_0_joint
- removed joint arm_1_joint
- removed joint arm_2_joint
- removed joint arm_3_joint
- removed joint arm_4_joint
- removed joint arm_5_joint
- removed joint base_joint
- added joint arm_left_joint: type revolute, parent base_link, child arm_left_link, origin xyz=0.0 0.0 0.0 rpy=0 0 0
- added joint arm_right_joint: type revolute, parent base_link, child arm_right_link, origin xyz=0.0 0.0 0.0 rpy=0 0 0

Commit message: fixed few error including namespace error. README still NOT ACCURATE./urdf_parser/src/pose.cpp

File: src/yamaro/output.urdf (robot description, URDF)
Before this commit: robot robot, 3 links, 2 joints
Links:
- removed link arm_left_link
- removed link arm_right_link
- added link part0_link, mass 10; collision sphere radius=1.0; visual sphere radius=1.0
Joints:
- removed joint arm_left_joint
- removed joint arm_right_joint
- added joint part0_joint: type fixed, parent root_link, child part0_link, origin xyz=0.0 0.0 0.0 rpy=0 0 0

Commit message: fixed more issues

File: src/yamaro/output.urdf (robot description, URDF)
Before this commit: robot drone, 2 links, 1 joints
Links:
- removed link part0_link
Joints:
- removed joint part0_joint
